File: usb_c_uart_debugger.kicad_sch (KiCad schematic)
At the start: 35 parts, among them J1 TYPE-C-31-M-12, J2 KH-2.54PH180-1X6P-L11.5, Q1 AO3401A, Q2 AO3401A, Q3 AO3400A, U1 CP2102N-A02-GQFN28R, U2 XC6206P332PR-G

Commit message: Advance the debugger to a routed, fabricable board
Place, generate and route the board, declare the pair as electrical paths
the toolkit measures on the copper, and install the fabrication outputs the
validated state produces.

The receptacle's four data terminals alternate along its land row, so the
two links that join each line's pair of terminals are non-planar: one of
them has to cross the other conductor on the back layer. That single fact
sets the launch geometry, the one layer change per conductor, and what the
plane under the pair is allowed to be missing. The design source names the
interruptions item by item and the layout prices them from the board's own
track width, via diameter, clearance and minimum pour width, so the
manifest's budget is arithmetic over that list rather than a tolerance.

The plane under the pair is closed to every other conductor for the whole
run, with windows only where the design source itself crosses it. The pair
is drawn with a vertex wherever a via or a pad meets it, so both meet end
on: copper landing part-way along a conductor would leave the meeting point
ambiguous over the width of the overlap, and the two plug orientations
could then only be compared approximately. They now measure exactly equal.

The bridge gets a board-owned land pattern. A stock QFN-28 footprint leaves
its thermal land unpasted and seals the pad ring, which would put the part's
only ground return behind a via in a pasted pad; this one pastes the land as
its datasheet's note requires and leaves the ring's corners open so the land
reaches the plane in copper.

Every applicable gate passes over the routed board: 27 PASS, 9 not
applicable, no failures and nothing unevaluated. release-check reports the
commit release-ready; no tag is created here.
Parts:
- U1: footprint Package_DFN_QFN:QFN-28-1EP_5x5mm_P0.5mm_EP3.25x3.25mm -> UsbCUartDebugger:QFN-28-1EP_5x5mm_P0.5mm_CP2102N
Changed lines of the file:
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@@
 		(property
 			"Footprint"
-			"Package_DFN_QFN:QFN-28-1EP_5x5mm_P0.5mm_EP3.25x3.25mm"
+			"UsbCUartDebugger:QFN-28-1EP_5x5mm_P0.5mm_CP2102N"
 			(at 736.6 165.1 0)
 			(hide yes)
